File: Design_blocks/SynthStuff.kicad_blocks/VC_Cross_Fader_SM.kicad_block/VC_Cross_Fader_SM.kicad_sch (KiCad schematic)
At the start: 47 parts, among them J1 Conn_01x08, J2 Conn_01x04, Q1 BC548, Q2 BC548, Q3 BC548, Q4 BC548, U1 TL074, U2 TL072

Commit message: Swapped XFader SM J1 and J2 refs around
Parts:
- renumbered J2 to J1, J1 to J2
Changed lines of the file:
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@@
 		(dnp no)
 		(fields_autoplaced yes)
-		(property "Reference" "J1"
+		(property "Reference" "J2"
 			(at 66.04 170.1799 0)
 			(show_name no)
@@
 			(project "DMH_Submodule_XFader"
 				(path "/58f4306d-5387-4983-bb08-41a2313fd315"
-					(reference "J1")
+					(reference "J2")
 					(unit 1)
 				)
@@
 		(in_pos_files yes)
 		(dnp no)
-		(property "Reference" "J2"
+		(property "Reference" "J1"
 			(at 35.56 201.9299 0)
 			(show_name no)
@@
 			(project "DMH_Submodule_XFader"
 				(path "/58f4306d-5387-4983-bb08-41a2313fd315"
-					(reference "J2")
+					(reference "J1")
 					(unit 1)
 				)

Commit message: Added solder jumpers to X faders
Parts:
- added C5: 33pF, Capacitor_THT:C_Disc_D3.0mm_W2.0mm_P2.50mm, symbol Device:C
- added JP1, JP2, JP3, JP4: SolderJumper_3_Open, Jumper:SolderJumper-3_P1.3mm_Open_RoundedPad1.0x1.5mm_NumberLabels, symbol Jumper:SolderJumper_3_Open
Connections:
- net at Q3.1 (C), R22.2: now also JP3.3 (B), JP4.1 (A); no longer R26.2
- net at Q4.1 (C), R23.2: now also JP3.1 (A), JP4.3 (B); no longer R25.2
- net at R18.1, R19.1, R21.1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: now also C5.1
- net at Q1.1 (C), R2.2: now also JP1.3 (B), JP2.1 (A); no longer R8.2
- net at Q2.1 (C), R3.2: now also JP1.1 (A), JP2.3 (B); no longer R7.2
- net CV Att In renamed CV_Att_In
- net CV Att Pot renamed CV_Att_Pot
- net CV Mix In renamed CV_Mix_In
- net In A renamed In_A
- net In B renamed In_B
- net Out A renamed Out_A
- net Out_A: no longer R21.2
- net Out B renamed Out_B
- net Out_B: now also R21.2
- net Out X renamed Out_X
- net Out_X: now also C5.2
- new net: JP2.2 (C), R8.2
- new net: JP3.2 (C), R25.2
- new net: JP1.2 (C), R7.2
- new net: JP4.2 (C), R26.2
Other:
- note added: "Optional"
- moved on the sheet: R26, R8
